Commit message: Revert "Merge request for changes to robot driver, teleop code and interface panels"

File: ur_description/urdf/ur5.urdf.xacro (robot description, xacro)
@@ -49,6 +49,5 @@
 		    <mesh filename="package://ur_description/meshes/ur5/visual/Base.dae" />
       </geometry>
-      <!-- <origin xyz="0.0 0.0 0.003" rpy="0.0 0.0 ${3.0 * pi / 4.0}" /> -->
-      <origin xyz="0.0 0.0 0.003" rpy="0.0 0.0 ${-pi/4.0}" />
+      <origin xyz="0.0 0.0 0.003" rpy="0.0 0.0 ${3.0 * pi / 4.0}" />
     </visual>
 	<collision>
@@ -66,6 +65,5 @@
     <parent link="${prefix}base_link" />
     <child link = "${prefix}shoulder_link" />
-    <!-- <origin xyz="0.0 0.0 ${shoulder_height}" rpy="0.0 0.0 0.0" /> -->
-    <origin xyz="0.0 0.0 ${shoulder_height}" rpy="0.0 0.0 3.1415" />
+    <origin xyz="0.0 0.0 ${shoulder_height}" rpy="0.0 0.0 0.0" />
     <axis xyz="0 0 1" />
     <limit lower="${-2.0 * pi}" upper="${2.0 * pi}" effort="150.0" velocity="${pi}"/>

Commit message: move marker around

File: ur_description/urdf/ur5.urdf.xacro (robot description, xacro)
@@ -226,4 +226,81 @@
   </joint>
   <link name="${prefix}ee_link" />
+  <link name="${prefix}gripper_link">
+    <visual>
+      <geometry>
+        <cylinder length="0.09" radius="0.065"/>
+      </geometry>
+      <origin rpy="0 0 0" xyz="0 0 0"/>
+      <material name="White"/>
+    </visual>
+    <visual>
+      <geometry>
+        <box size="0.15 0.02 0.05"/>
+      </geometry>
+      <origin rpy="0 0 0" xyz="0 -0.01 0.065"/>
+    </visual>
+    <visual>
+      <geometry>
+        <box size="0.03 0.02 0.07"/>
+      </geometry>
+      <origin rpy="0 0 0" xyz="-0.06 -0.01 0.125"/>
+    </visual>
+    <visual>
+      <geometry>
+        <box size="0.03 0.02 0.07"/>
+      </geometry>
+      <origin rpy="0 0 0" xyz="0.06 -0.01 0.125"/>
+    </visual>
+    <collision>
+      <geometry>
+        <cylinder length="0.09" radius="0.065"/>
+      </geometry>
+      <origin rpy="0 0 0" xyz="0 0 0"/>
+    </collision>
+    <collision>
+      <geometry>
+        <box size="0.15 0.02 0.05"/>
+      </geometry>
+      <origin rpy="0 0 0" xyz="0 -0.01 0.065"/>
+    </collision>
+    <collision>
+      <geometry>
+        <box size="0.03 0.02 0.07"/>
+      </geometry>
+      <origin rpy="0 0 0" xyz="-0.06 -0.01 0.125"/>
+    </collision>
+    <collision>
+      <geometry>
+        <box size="0.03 0.02 0.07"/>
+      </geometry>
+      <origin rpy="0 0 0" xyz="0.06 -0.01 0.125"/>
+    </collision>
+  </link>
+  <joint name="${prefix}ee_link_gripper" type="fixed">
+    <parent link="${prefix}ee_link"/>
+    <child link="${prefix}gripper_link"/>
+    <origin rpy="${pi/2} ${pi/2} ${pi/2}" xyz="0.05 0 0"/>
+  </joint>
+  <link name="${prefix}marker_link">
+    <visual>
+      <geometry>
+        <box size="0.102 0.045 0.102"/>
+      </geometry>
+      <origin rpy="0 0 0" xyz="-0.01 0.09 0"/>
+      <material name="LightGrey"/>
+    </visual>
+    <collision>
+      <geometry>
+        <box size="0.102 0.045 0.102"/>
+      </geometry>
+      <origin rpy="0 0 0" xyz="-0.01 0.09 0"/>
+    </collision>
+  </link>
+  <joint name="${prefix}ee_link_marker" type="fixed">
+    <parent link="${prefix}ee_link"/>
+    <child link="${prefix}marker_link"/>
+    <!-- <origin rpy="-1.1579458160307363 -1.558725130964142 -0.47951188571736364" xyz="-0.0131988 0.105739 -0.0014977"/> -->
+    <origin rpy="0 0 0" xyz="0 0 0"/>
+  </joint>
   <!-- Change to fix urdf_parse_error -->
   <!-- <xacro:ur5_arm_transmission prefix="${prefix}" /> -->

File: ur_description/urdf/ur5_joint_limited.urdf.xacro (robot description, xacro)
@@ -236,22 +236,19 @@
     <visual>
       <geometry>
-        <box size="0.15 0.02 0.04"/>
-      </geometry>
-      <origin rpy="0 0 0" xyz="0 0 0.065"/>
-      <material name="LightGrey"/>
-    </visual>
-    <visual>
-      <geometry>
-        <box size="0.03 0.02 0.05"/>
-      </geometry>
-      <origin rpy="0 0 0" xyz="-0.06 0 0.11"/>
-      <material name="White"/>
-    </visual>
-    <visual>
-      <geometry>
-        <box size="0.03 0.02 0.05"/>
-      </geometry>
-      <origin rpy="0 0 0" xyz="0.06 0 0.11"/>
-      <material name="White"/>
+        <box size="0.15 0.02 0.05"/>
+      </geometry>
+      <origin rpy="0 0 0" xyz="0 -0.01 0.065"/>
+    </visual>
+    <visual>
+      <geometry>
+        <box size="0.03 0.02 0.07"/>
+      </geometry>
+      <origin rpy="0 0 0" xyz="-0.06 -0.01 0.125"/>
+    </visual>
+    <visual>
+      <geometry>
+        <box size="0.03 0.02 0.07"/>
+      </geometry>
+      <origin rpy="0 0 0" xyz="0.06 -0.01 0.125"/>
     </visual>
     <collision>
@@ -263,19 +260,19 @@
     <collision>
       <geometry>
-        <box size="0.15 0.02 0.04"/>
-      </geometry>
-      <origin rpy="0 0 0" xyz="0 0 0.065"/>
-    </collision>
-    <collision>
-      <geometry>
-        <box size="0.03 0.02 0.05"/>
-      </geometry>
-      <origin rpy="0 0 0" xyz="-0.06 0 0.11"/>
-    </collision>
-    <collision>
-      <geometry>
-        <box size="0.03 0.02 0.05"/>
-      </geometry>
-      <origin rpy="0 0 0" xyz="0.06 0 0.11"/>
+        <box size="0.15 0.02 0.05"/>
+      </geometry>
+      <origin rpy="0 0 0" xyz="0 -0.01 0.065"/>
+    </collision>
+    <collision>
+      <geometry>
+        <box size="0.03 0.02 0.07"/>
+      </geometry>
+      <origin rpy="0 0 0" xyz="-0.06 -0.01 0.125"/>
+    </collision>
+    <collision>
+      <geometry>
+        <box size="0.03 0.02 0.07"/>
+      </geometry>
+      <origin rpy="0 0 0" xyz="0.06 -0.01 0.125"/>
     </collision>
   </link>
@@ -284,4 +281,25 @@
     <child link="${prefix}gripper_link"/>
     <origin rpy="${pi/2} ${pi/2} ${pi/2}" xyz="0.05 0 0"/>
+  </joint>
+  <link name="${prefix}marker_link">
+    <visual>
+      <geometry>
+        <box size="0.102 0.045 0.102"/>
+      </geometry>
+      <origin rpy="0 0 0" xyz="0.07 0.09 0"/>
+      <material name="LightGrey"/>
+    </visual>
+    <collision>
+      <geometry>
+        <box size="0.102 0.045 0.102"/>
+      </geometry>
+      <origin rpy="0 0 0" xyz="0.05 0.09 0"/>
+    </collision>
+  </link>
+  <joint name="${prefix}ee_link_marker" type="fixed">
+    <parent link="${prefix}ee_link"/>
+    <child link="${prefix}marker_link"/>
+    <!-- <origin rpy="-1.1579458160307363 -1.558725130964142 -0.47951188571736364" xyz="-0.0131988 0.105739 -0.0014977"/> -->
+    <origin rpy="0 0 0" xyz="0 0 0"/>
   </joint>
   <!-- Change to fix urdf_parse_error -->

Commit message: tweaks to config for our ur5

File: ur_description/urdf/ur5.urdf.xacro (robot description, xacro)
@@ -266,13 +266,13 @@
     <collision>
       <geometry>
-        <box size="0.03 0.02 0.07"/>
-      </geometry>
-      <origin rpy="0 0 0" xyz="-0.06 -0.01 0.125"/>
-    </collision>
-    <collision>
-      <geometry>
-        <box size="0.03 0.02 0.07"/>
-      </geometry>
-      <origin rpy="0 0 0" xyz="0.06 -0.01 0.125"/>
+        <box size="0.06 0.04 0.08"/>
+      </geometry>
+      <origin rpy="0 0 0" xyz="-0.05 -0.01 0.125"/>
+    </collision>
+    <collision>
+      <geometry>
+        <box size="0.06 0.04 0.08"/>
+      </geometry>
+      <origin rpy="0 0 0" xyz="0.05 -0.01 0.125"/>
     </collision>
   </link>

File: ur_description/urdf/ur5_joint_limited.urdf.xacro (robot description, xacro)
@@ -242,5 +242,5 @@
     <visual>
       <geometry>
-        <box size="0.03 0.02 0.07"/>
+        <box size="0.04 0.03 0.08"/>
       </geometry>
       <origin rpy="0 0 0" xyz="-0.06 -0.01 0.125"/>
@@ -248,5 +248,5 @@
     <visual>
       <geometry>
-        <box size="0.03 0.02 0.07"/>
+        <box size="0.04 0.03 0.08"/>
       </geometry>
       <origin rpy="0 0 0" xyz="0.06 -0.01 0.125"/>
@@ -266,13 +266,13 @@
     <collision>
       <geometry>
-        <box size="0.03 0.02 0.07"/>
-      </geometry>
-      <origin rpy="0 0 0" xyz="-0.06 -0.01 0.125"/>
-    </collision>
-    <collision>
-      <geometry>
-        <box size="0.03 0.02 0.07"/>
-      </geometry>
-      <origin rpy="0 0 0" xyz="0.06 -0.01 0.125"/>
+        <box size="0.06 0.04 0.08"/>
+      </geometry>
+      <origin rpy="0 0 0" xyz="-0.05 -0.01 0.125"/>
+    </collision>
+    <collision>
+      <geometry>
+        <box size="0.06 0.04 0.08"/>
+      </geometry>
+      <origin rpy="0 0 0" xyz="0.05 -0.01 0.125"/>
     </collision>
   </link>

Commit message: assorted updates

File: ur_description/urdf/ur5.urdf.xacro (robot description, xacro)
@@ -236,19 +236,25 @@
     <visual>
       <geometry>
+        <box size="0.05 0.075 0.125"/>
+      </geometry>
+      <origin rpy="0 0 0" xyz="-0.10 -0.01 0.0"/>
+    </visual>
+    <visual>
+      <geometry>
         <box size="0.15 0.02 0.05"/>
       </geometry>
-      <origin rpy="0 0 0" xyz="0 -0.01 0.065"/>
-    </visual>
-    <visual>
-      <geometry>
-        <box size="0.03 0.02 0.07"/>
-      </geometry>
-      <origin rpy="0 0 0" xyz="-0.06 -0.01 0.125"/>
-    </visual>
-    <visual>
-      <geometry>
-        <box size="0.03 0.02 0.07"/>
-      </geometry>
-      <origin rpy="0 0 0" xyz="0.06 -0.01 0.125"/>
+      <origin rpy="0 0 0" xyz="0.0 -0.01 0.065"/>
+    </visual>
+    <visual>
+      <geometry>
+        <box size="0.04 0.03 0.055"/>
+      </geometry>
+      <origin rpy="0 0 0" xyz="-0.06 -0.01 0.110"/>
+    </visual>
+    <visual>
+      <geometry>
+        <box size="0.04 0.03 0.055"/>
+      </geometry>
+      <origin rpy="0 0 0" xyz="0.06 -0.01 0.110"/>
     </visual>
     <collision>
@@ -260,19 +266,26 @@
     <collision>
       <geometry>
+        <box size="0.05 0.075 0.125"/>
+      </geometry>
+      <origin rpy="0 0 0" xyz="-0.10 -0.01 0.0"/>
+    </collision>
+    <collision>
+      <geometry>
         <box size="0.15 0.02 0.05"/>
       </geometry>
-      <origin rpy="0 0 0" xyz="0 -0.01 0.065"/>
-    </collision>
-    <collision>
-      <geometry>
-        <box size="0.06 0.04 0.08"/>
-      </geometry>
-      <origin rpy="0 0 0" xyz="-0.05 -0.01 0.125"/>
-    </collision>
-    <collision>
-      <geometry>
-        <box size="0.06 0.04 0.08"/>
-      </geometry>
-      <origin rpy="0 0 0" xyz="0.05 -0.01 0.125"/>
+      <origin rpy="0 0 0" xyz="0.0 -0.01 0.065"/>
+    </collision>
+    <!-- Simplified Robotiq S Model Gripper fingers for faster collision checks -->
+    <collision>
+      <geometry>
+        <box size="0.04 0.03 0.08"/>
+      </geometry>
+      <origin rpy="0 0 0" xyz="-0.06 -0.01 0.110"/>
+    </collision>
+    <collision>
+      <geometry>
+        <box size="0.04 0.03 0.08"/>
+      </geometry>
+      <origin rpy="0 0 0" xyz="0.06 -0.01 0.110"/>
     </collision>
   </link>
@@ -280,5 +293,5 @@
     <parent link="${prefix}ee_link"/>
     <child link="${prefix}gripper_link"/>
-    <origin rpy="${pi/2} ${pi/2} ${pi/2}" xyz="0.05 0 0"/>
+    <origin rpy="${pi/2} ${pi/2} ${pi/2}" xyz="0.05 0 -0.01"/>
   </joint>
   <link name="${prefix}marker_link">

File: ur_description/urdf/ur5_joint_limited.urdf.xacro (robot description, xacro)
@@ -236,19 +236,25 @@
     <visual>
       <geometry>
+        <box size="0.05 0.05 0.125"/>
+      </geometry>
+      <origin rpy="0 0 0" xyz="-0.08 0 0.0"/>
+    </visual>
+    <visual>
+      <geometry>
         <box size="0.15 0.02 0.05"/>
       </geometry>
-      <origin rpy="0 0 0" xyz="0 -0.01 0.065"/>
-    </visual>
-    <visual>
-      <geometry>
-        <box size="0.04 0.03 0.08"/>
-      </geometry>
-      <origin rpy="0 0 0" xyz="-0.06 -0.01 0.125"/>
-    </visual>
-    <visual>
-      <geometry>
-        <box size="0.04 0.03 0.08"/>
-      </geometry>
-      <origin rpy="0 0 0" xyz="0.06 -0.01 0.125"/>
+      <origin rpy="0 0 0" xyz="0.0 -0.01 0.065"/>
+    </visual>
+    <visual>
+      <geometry>
+        <box size="0.04 0.03 0.055"/>
+      </geometry>
+      <origin rpy="0 0 0" xyz="-0.06 -0.01 0.110"/>
+    </visual>
+    <visual>
+      <geometry>
+        <box size="0.04 0.03 0.055"/>
+      </geometry>
+      <origin rpy="0 0 0" xyz="0.06 -0.01 0.110"/>
     </visual>
     <collision>
@@ -260,19 +266,25 @@
     <collision>
       <geometry>
+        <box size="0.05 0.075 0.125"/>
+      </geometry>
+      <origin rpy="0 0 0" xyz="-0.10 -0.01 0.0"/>
+    </collision>
+    <collision>
+      <geometry>
         <box size="0.15 0.02 0.05"/>
       </geometry>
-      <origin rpy="0 0 0" xyz="0 -0.01 0.065"/>
-    </collision>
-    <collision>
-      <geometry>
-        <box size="0.06 0.04 0.08"/>
-      </geometry>
-      <origin rpy="0 0 0" xyz="-0.05 -0.01 0.125"/>
-    </collision>
-    <collision>
-      <geometry>
-        <box size="0.06 0.04 0.08"/>
-      </geometry>
-      <origin rpy="0 0 0" xyz="0.05 -0.01 0.125"/>
+      <origin rpy="0 0 0" xyz="0.0 -0.01 0.065"/>
+    </collision>
+    <collision>
+      <geometry>
+        <box size="0.04 0.03 0.055"/>
+      </geometry>
+      <origin rpy="0 0 0" xyz="-0.06 -0.01 0.110"/>
+    </collision>
+    <collision>
+      <geometry>
+        <box size="0.04 0.03 0.055"/>
+      </geometry>
+      <origin rpy="0 0 0" xyz="0.06 -0.01 0.110"/>
     </collision>
   </link>
@@ -280,5 +292,5 @@
     <parent link="${prefix}ee_link"/>
     <child link="${prefix}gripper_link"/>
-    <origin rpy="${pi/2} ${pi/2} ${pi/2}" xyz="0.05 0 0"/>
+    <origin rpy="${pi/2} ${pi/2} ${pi/2}" xyz="0.05 0 -0.01"/>
   </joint>
   <link name="${prefix}marker_link">

Commit message: enlarging the fingers

File: ur_description/urdf/ur5.urdf.xacro (robot description, xacro)
@@ -246,7 +246,8 @@
       <origin rpy="0 0 0" xyz="0.0 -0.01 0.065"/>
     </visual>
-    <visual>
-      <geometry>
-        <box size="0.04 0.03 0.055"/>
+    <!-- Simplified Robotiq S Model Gripper fingers for faster collision checks, non-limited joint angles -->
+    <visual>
+      <geometry>
+        <box size="0.04 0.03 0.08"/>
       </geometry>
       <origin rpy="0 0 0" xyz="-0.06 -0.01 0.110"/>
@@ -254,5 +255,5 @@
     <visual>
       <geometry>
-        <box size="0.04 0.03 0.055"/>
+        <box size="0.04 0.03 0.08"/>
       </geometry>
       <origin rpy="0 0 0" xyz="0.06 -0.01 0.110"/>

File: ur_description/urdf/ur5_joint_limited.urdf.xacro (robot description, xacro)
@@ -247,14 +247,16 @@
     </visual>
     <visual>
-      <geometry>
-        <box size="0.04 0.03 0.055"/>
-      </geometry>
-      <origin rpy="0 0 0" xyz="-0.06 -0.01 0.110"/>
-    </visual>
-    <visual>
-      <geometry>
-        <box size="0.04 0.03 0.055"/>
-      </geometry>
-      <origin rpy="0 0 0" xyz="0.06 -0.01 0.110"/>
+      <!-- Simplified Robotiq S Model Gripper fingers for faster collision checks, limited joint angles -->
+      <!-- z size = 0.08, z origin = 0.12 is pretty accurate -->
+      <geometry>
+        <box size="0.04 0.03 0.09"/>
+      </geometry>
+      <origin rpy="0 0 0" xyz="-0.06 -0.01 0.125"/>
+    </visual>
+    <visual>
+      <geometry>
+        <box size="0.04 0.03 0.09"/>
+      </geometry>
+      <origin rpy="0 0 0" xyz="0.06 -0.01 0.125"/>
     </visual>
     <collision>
@@ -276,15 +278,16 @@
       <origin rpy="0 0 0" xyz="0.0 -0.01 0.065"/>
     </collision>
-    <collision>
-      <geometry>
-        <box size="0.04 0.03 0.055"/>
-      </geometry>
-      <origin rpy="0 0 0" xyz="-0.06 -0.01 0.110"/>
-    </collision>
-    <collision>
-      <geometry>
-        <box size="0.04 0.03 0.055"/>
-      </geometry>
-      <origin rpy="0 0 0" xyz="0.06 -0.01 0.110"/>
+    <!-- Simplified Robotiq S Model Gripper fingers for faster collision checks, limited joint angles -->
+    <collision>
+      <geometry>
+        <box size="0.04 0.03 0.09"/>
+      </geometry>
+      <origin rpy="0 0 0" xyz="-0.06 -0.01 0.125"/>
+    </collision>
+    <collision>
+      <geometry>
+        <box size="0.04 0.03 0.09"/>
+      </geometry>
+      <origin rpy="0 0 0" xyz="0.06 -0.01 0.125"/>
     </collision>
   </link>
