Commit message: Make urdf match our current marker position

File: ur_description/urdf/ur5_joint_limited.urdf.xacro (robot description, xacro)
@@ -287,5 +287,5 @@
         <box size="0.102 0.045 0.102"/>
       </geometry>
-      <origin rpy="0 0 0" xyz="0.07 0.09 0"/>
+      <origin rpy="0 0 0" xyz="0.02 0.09 0"/>
       <material name="LightGrey"/>
     </visual>
@@ -294,5 +294,5 @@
         <box size="0.102 0.045 0.102"/>
       </geometry>
-      <origin rpy="0 0 0" xyz="0.05 0.09 0"/>
+      <origin rpy="0 0 0" xyz="0.02 0.09 0"/>
     </collision>
   </link>

Commit message: ur5_joint_limited.urdf.xacro update marker link size and position

File: ur_description/urdf/ur5_joint_limited.urdf.xacro (robot description, xacro)
@@ -4,4 +4,8 @@
   <xacro:include filename="$(find ur_description)/urdf/ur5.gazebo.xacro" />
   <xacro:include filename="$(find ur_description)/urdf/materials.urdf.xacro" />
+<!--
+This is the file typically used to define the simulated robot model utilized while
+costar is run on a real robot.
+-->
 <!--
 DH for UR5:
@@ -297,10 +301,16 @@
     <origin rpy="${pi/2} ${pi/2} ${pi/2}" xyz="0.05 0 -0.01"/>
   </joint>
+  <!-- Link and box for the ar tag marker panel on the gripper -->
   <link name="${prefix}marker_link">
     <visual>
       <geometry>
-        <box size="0.102 0.045 0.102"/>
-      </geometry>
-      <origin rpy="0 0 0" xyz="0.02 0.09 0"/>
+        <!-- width thickness height -->
+        <box size="0.115 0.045 0.11"/>
+      </geometry>
+      <!-- +x is towards the gripper tip parallel to the marker
+           -y is towards the center of the gripper, normal to the marker
+           +z moves left and right
+           -->
+      <origin rpy="0 0 0" xyz="0.01 0.09 0"/>
       <material name="LightGrey"/>
     </visual>
